Commit message: feat: replace primitive URDF with proper KR6 R700 STL/DAE meshes from ROS-Industrial + full refueling mission

File: kuka_refuel_ws/src/kuka_kr6_gazebo/urdf/kr6_r700_2_clean.urdf (robot description, URDF)
Before this commit: robot kr6_r700_2, 11 links, 10 joints
Links:
- removed link base
- removed link flange
- removed link tool0
- removed link world
- link base_link: mass 1.6916E1 -> 5.0; geometry collision mesh filename=package://kuka_kr6_gazebo/meshes/collision/base_link.stl; visual mesh filename=package://kuka_kr6_gazebo/meshes/visual/base_link.dae
- link link_1: mass 8.416E0 -> 4.0; geometry collision mesh filename=package://kuka_kr6_gazebo/meshes/collision/link_1.stl; visual mesh filename=package://kuka_kr6_gazebo/meshes/visual/link_1.dae
- link link_2: mass 1.55659E1 -> 3.5; geometry collision mesh filename=package://kuka_kr6_gazebo/meshes/collision/link_2.stl; visual mesh filename=package://kuka_kr6_gazebo/meshes/visual/link_2.dae
- link link_3: mass 5.303E0 -> 2.5; geometry collision mesh filename=package://kuka_kr6_gazebo/meshes/collision/link_3.stl; visual mesh filename=package://kuka_kr6_gazebo/meshes/visual/link_3.dae
- link link_4: mass 4.6129999999999995E0 -> 2.0; geometry collision mesh filename=package://kuka_kr6_gazebo/meshes/collision/link_4.stl; visual mesh filename=package://kuka_kr6_gazebo/meshes/visual/link_4.dae
- link link_5: mass 1.6128E0 -> 1.0; geometry collision mesh filename=package://kuka_kr6_gazebo/meshes/collision/link_5.stl; visual mesh filename=package://kuka_kr6_gazebo/meshes/visual/link_5.dae
- link link_6: mass 7.34E-1 -> 0.5; geometry collision mesh filename=package://kuka_kr6_gazebo/meshes/collision/link_6.stl; visual mesh filename=package://kuka_kr6_gazebo/meshes/visual/link_6.dae
Joints:
- removed joint base_link-base
- removed joint link6-flange
- removed joint link6-tool0
- removed joint world-base_link
- joint joint_1: axis 0.0 0.0 1.0 -> 0 0 -1; limit lower=-2.967059725E0 upper=2.967059725E0 effort=1.86E2 velocity=6.2831853071795862E0 -> lower=-2.967059725 upper=2.967059725 effort=100 velocity=6.2832; origin xyz=0.0 0.0 0.20800000000000002 rpy=3.141592653589793 -0.0 0.0 -> xyz=0 0 0.4 rpy=0 0 0
- joint joint_2: axis 0.0 0.0 1.0 -> 0 1 0; limit lower=-3.316125575E0 upper=7.853981625E-1 effort=1.6893729997505432E2 velocity=5.2359877559829888E0 -> lower=-3.316125575 upper=0.785398163 effort=100 velocity=5.2360; origin xyz=0.025 -0.0907 -0.192 rpy=1.5707963267948966 -0.0 0.0 -> xyz=0.025 0 0 rpy=0 0 0
- joint joint_3: axis 0.0 0.0 1.0 -> 0 1 0; limit lower=-2.0943951E0 upper=2.72271363E0 effort=8.1493186258254326E1 velocity=6.2831853071795862E0 -> lower=-2.094395100 upper=2.722713630 effort=100 velocity=6.2832; origin xyz=0.335 0.0 -0.004200000000000001 rpy=0.0 -0.0 0.0 -> xyz=0.315 0 0 rpy=0 0 0
- joint joint_4: axis 0.0 0.0 1.0 -> -1 0 0; limit lower=-3.2288591125E0 upper=3.2288591125E0 effort=4.8879867848304357E1 velocity=7.8539816339744828E0 -> lower=-3.228859113 upper=3.228859113 effort=100 velocity=6.6497; origin xyz=0.14100000000000001 -0.025 -0.08650000000000001 rpy=1.5707963267948966 -0.0 -1.5707963267948966 -> xyz=0 0 0.035 rpy=0 0 0
- joint joint_5: axis 0.0 0.0 1.0 -> 0 1 0; limit lower=-2.0943951E0 upper=2.0943951E0 effort=4.0135638235238289E1 velocity=7.8539816339744828E0 -> lower=-2.094395100 upper=2.094395100 effort=100 velocity=6.7720; origin xyz=0.0 0.0505 -0.224 rpy=0.0 1.5707963267948966 1.5707963267948966 -> xyz=0.365 0 0 rpy=0 0 0
- joint joint_6: axis 0.0 0.0 1.0 -> -1 0 0; limit lower=-6.108652375E0 upper=6.108652375E0 effort=2.7358196129032258E1 velocity=9.42477796076938E0 -> lower=-6.108652375 upper=6.108652375 effort=100 velocity=10.7338; origin xyz=0.0615 0.0 -0.0505 rpy=1.5707963267948966 -0.0 -1.5707963267948966 -> xyz=0.080 0 0 rpy=0 0 0

Commit message: fix: realistic inertials from KUKA datasheet, PID gains, joint damping/friction for Gazebo stability

File: kuka_refuel_ws/src/kuka_kr6_gazebo/urdf/kr6_r700_2_clean.urdf (robot description, URDF)
Before this commit: robot kr6_r700, 8 links, 7 joints
Links:
- link base_link: mass 5.0 -> 15.0
- link link_1: mass 4.0 -> 12.0
- link link_2: mass 3.5 -> 10.0
- link link_3: mass 2.5 -> 5.0
- link link_4: mass 2.0 -> 4.0
- link link_5: mass 1.0 -> 2.0
- link link_6: mass 0.5 -> 1.0
Joints:
- joint joint_1: limit lower=-2.967059725 upper=2.967059725 effort=100 velocity=6.2832 -> lower=-2.967059725 upper=2.967059725 effort=200 velocity=6.2832
- joint joint_2: limit lower=-3.316125575 upper=0.785398163 effort=100 velocity=5.2360 -> lower=-3.316125575 upper=0.785398163 effort=200 velocity=5.2360
- joint joint_3: limit lower=-2.094395100 upper=2.722713630 effort=100 velocity=6.2832 -> lower=-2.094395100 upper=2.722713630 effort=200 velocity=6.2832
- joint joint_6: limit lower=-6.108652375 upper=6.108652375 effort=100 velocity=10.7338 -> lower=-6.108652375 upper=6.108652375 effort=50 velocity=10.7338
