Commit message: feat: convert entire ROS package from ROS 2 to ROS Noetic (catkin, gazebo_ros_control, XML launch)

File: kuka_refuel_ws/src/kuka_kr6_gazebo/urdf/kr6_r700.gazebo.xacro (robot description, xacro)
@@ -3,33 +3,30 @@
   <!-- Include the raw clean URDF (primitive cylinders/boxes) -->
   <xacro:include filename="$(find kuka_kr6_gazebo)/urdf/kr6_r700_clean.urdf" />
-  <!-- ROS 2 Control tag for Gazebo -->
-  <ros2_control name="GazeboSystem" type="system">
-    <hardware>
-      <plugin>gazebo_ros2_control/GazeboSystem</plugin>
-    </hardware>
-    <xacro:macro name="kuka_joint_control" params="joint_name">
-      <joint name="${joint_name}">
-        <command_interface name="position">
-          <param name="min">-3.14</param>
-          <param name="max">3.14</param>
-        </command_interface>
-        <state_interface name="position"/>
-        <state_interface name="velocity"/>
-        <state_interface name="effort"/>
-      </joint>
-    </xacro:macro>
-    <xacro:kuka_joint_control joint_name="joint_1"/>
-    <xacro:kuka_joint_control joint_name="joint_2"/>
-    <xacro:kuka_joint_control joint_name="joint_3"/>
-    <xacro:kuka_joint_control joint_name="joint_4"/>
-    <xacro:kuka_joint_control joint_name="joint_5"/>
-    <xacro:kuka_joint_control joint_name="joint_6"/>
-  </ros2_control>
-  <!-- Gazebo ROS 2 Control Plugin -->
+  <!-- Gazebo ROS Control Plugin (Noetic) -->
   <gazebo>
-    <plugin filename="libgazebo_ros2_control.so" name="gazebo_ros2_control">
-      <parameters>$(find kuka_kr6_gazebo)/config/ros2_controllers.yaml</parameters>
+    <plugin name="gazebo_ros_control" filename="libgazebo_ros_control.so">
+      <robotNamespace>/</robotNamespace>
+      <robotSimType>gazebo_ros_control/DefaultRobotHWSim</robotSimType>
     </plugin>
   </gazebo>
+  <!-- Transmission for each joint (required for gazebo_ros_control) -->
+  <xacro:macro name="kuka_transmission" params="joint_name">
+    <transmission name="${joint_name}_trans">
+      <type>transmission_interface/SimpleTransmission</type>
+      <joint name="${joint_name}">
+        <hardwareInterface>hardware_interface/PositionJointInterface</hardwareInterface>
+      </joint>
+      <actuator name="${joint_name}_actuator">
+        <hardwareInterface>hardware_interface/PositionJointInterface</hardwareInterface>
+        <mechanicalReduction>1</mechanicalReduction>
+      </actuator>
+    </transmission>
+  </xacro:macro>
+  <xacro:kuka_transmission joint_name="joint_1"/>
+  <xacro:kuka_transmission joint_name="joint_2"/>
+  <xacro:kuka_transmission joint_name="joint_3"/>
+  <xacro:kuka_transmission joint_name="joint_4"/>
+  <xacro:kuka_transmission joint_name="joint_5"/>
+  <xacro:kuka_transmission joint_name="joint_6"/>
   <!-- Physics materials -->
   <gazebo reference="base_link">

Commit message: feat: migrate full ROS stack from Noetic to ROS2 Humble
- Build system: catkin → ament_cmake across all 3 packages
  (kuka_kr6_gazebo, ur5_gazebo, ur_description)
- URDF/Xacro: replaced gazebo_ros_control + transmission_interface
  with ros2_control hardware interface + gazebo_ros2_control plugin
  for both KUKA KR6 R700 and UR5
- Controller config: new ur5_ros2_controllers.yaml for UR5;
  KUKA ros2_controllers.yaml was already present
- Launch: 5 XML .launch files → 4 Python .launch.py files
  (gazebo.launch.py, rviz.launch.py, ur5_refuel.launch.py,
  ur5_rviz.launch.py)
- Python nodes: rospy/actionlib → rclpy/action in refuel_mission.py,
  admittance_node.py (full Node subclass rewrite), car_model.py
  (SpawnModel → SpawnEntity)
- All ROS1 files preserved in deprecated/ros1_build/ and
  deprecated/ros1_launch/ — nothing deleted
- Pure-Python planning stack (IK, STOMP, Bubble Strips) untouched
- Updated README and self_contribution_audit.md

File: kuka_refuel_ws/src/kuka_kr6_gazebo/urdf/kr6_r700.gazebo.xacro (robot description, xacro)
@@ -3,30 +3,67 @@
   <!-- Include the raw clean URDF (primitive cylinders/boxes) -->
   <xacro:include filename="$(find kuka_kr6_gazebo)/urdf/kr6_r700_2_clean.urdf" />
-  <!-- Gazebo ROS Control Plugin (Noetic) -->
+  <!-- ================================================================
+       ROS2 Control Hardware Interface (replaces gazebo_ros_control +
+       transmission_interface from ROS1 — see deprecated/ros1_build/)
+       ================================================================ -->
+  <ros2_control name="GazeboSystem" type="system">
+    <hardware>
+      <plugin>gazebo_ros2_control/GazeboSystem</plugin>
+    </hardware>
+    <joint name="joint_1">
+      <command_interface name="position">
+        <param name="min">-2.9671</param>  <!-- -170 deg -->
+        <param name="max">2.9671</param>   <!--  170 deg -->
+      </command_interface>
+      <state_interface name="position"/>
+      <state_interface name="velocity"/>
+    </joint>
+    <joint name="joint_2">
+      <command_interface name="position">
+        <param name="min">-3.3161</param>  <!-- -190 deg -->
+        <param name="max">0.7854</param>   <!--   45 deg -->
+      </command_interface>
+      <state_interface name="position"/>
+      <state_interface name="velocity"/>
+    </joint>
+    <joint name="joint_3">
+      <command_interface name="position">
+        <param name="min">-2.0944</param>  <!-- -120 deg -->
+        <param name="max">2.7227</param>   <!--  156 deg -->
+      </command_interface>
+      <state_interface name="position"/>
+      <state_interface name="velocity"/>
+    </joint>
+    <joint name="joint_4">
+      <command_interface name="position">
+        <param name="min">-3.2289</param>  <!-- -185 deg -->
+        <param name="max">3.2289</param>   <!--  185 deg -->
+      </command_interface>
+      <state_interface name="position"/>
+      <state_interface name="velocity"/>
+    </joint>
+    <joint name="joint_5">
+      <command_interface name="position">
+        <param name="min">-2.0944</param>  <!-- -120 deg -->
+        <param name="max">2.0944</param>   <!--  120 deg -->
+      </command_interface>
+      <state_interface name="position"/>
+      <state_interface name="velocity"/>
+    </joint>
+    <joint name="joint_6">
+      <command_interface name="position">
+        <param name="min">-6.1087</param>  <!-- -350 deg -->
+        <param name="max">6.1087</param>   <!--  350 deg -->
+      </command_interface>
+      <state_interface name="position"/>
+      <state_interface name="velocity"/>
+    </joint>
+  </ros2_control>
+  <!-- gazebo_ros2_control plugin (replaces libgazebo_ros_control.so from ROS1) -->
   <gazebo>
-    <plugin name="gazebo_ros_control" filename="libgazebo_ros_control.so">
-      <robotNamespace>/</robotNamespace>
-      <robotSimType>gazebo_ros_control/DefaultRobotHWSim</robotSimType>
+    <plugin name="gazebo_ros2_control" filename="libgazebo_ros2_control.so">
+      <parameters>$(find kuka_kr6_gazebo)/config/ros2_controllers.yaml</parameters>
     </plugin>
   </gazebo>
-  <!-- Transmission for each joint (required for gazebo_ros_control) -->
-  <xacro:macro name="kuka_transmission" params="joint_name">
-    <transmission name="${joint_name}_trans">
-      <type>transmission_interface/SimpleTransmission</type>
-      <joint name="${joint_name}">
-        <hardwareInterface>hardware_interface/PositionJointInterface</hardwareInterface>
-      </joint>
-      <actuator name="${joint_name}_actuator">
-        <hardwareInterface>hardware_interface/PositionJointInterface</hardwareInterface>
-        <mechanicalReduction>1</mechanicalReduction>
-      </actuator>
-    </transmission>
-  </xacro:macro>
-  <xacro:kuka_transmission joint_name="joint_1"/>
-  <xacro:kuka_transmission joint_name="joint_2"/>
-  <xacro:kuka_transmission joint_name="joint_3"/>
-  <xacro:kuka_transmission joint_name="joint_4"/>
-  <xacro:kuka_transmission joint_name="joint_5"/>
-  <xacro:kuka_transmission joint_name="joint_6"/>
   <!-- Physics materials -->
   <gazebo reference="base_link">

Commit message: feat: migrate from Gazebo Classic to Gz Sim (ROS2 Jazzy)
- Replace gazebo_ros with ros_gz_sim in all package.xml and launch files
- Replace gazebo_ros2_control with gz_ros2_control in URDFs/xacro
  (GazeboSystem → GzSimSystem, libgazebo_ros2_control.so → gz_ros2_control-system)
- Rewrite world file as SDF 1.9 with explicit Gz Sim system plugins
- Replace spawn_entity.py with ros_gz_sim create in launch files
- Replace gazebo_msgs.srv.SpawnEntity with subprocess ros_gz_sim create
  in car_model.py and refuel_mission.py
- Replace Gazebo/Orange named materials with explicit RGBA values
- Comment out UR5 FT sensor plugin (no Gz Sim equivalent yet)
- Move old world file to deprecated/ros1_build/

File: kuka_refuel_ws/src/kuka_kr6_gazebo/urdf/kr6_r700.gazebo.xacro (robot description, xacro)
@@ -7,7 +7,7 @@
        transmission_interface from ROS1 — see deprecated/ros1_build/)
        ================================================================ -->
-  <ros2_control name="GazeboSystem" type="system">
+  <ros2_control name="GzSimSystem" type="system">
     <hardware>
-      <plugin>gazebo_ros2_control/GazeboSystem</plugin>
+      <plugin>gz_ros2_control/GzSimSystem</plugin>
     </hardware>
     <joint name="joint_1">
@@ -60,8 +60,8 @@
     </joint>
   </ros2_control>
-  <!-- gazebo_ros2_control plugin (replaces libgazebo_ros_control.so from ROS1) -->
+  <!-- gz_ros2_control plugin for Gz Sim (Gazebo Harmonic) -->
   <xacro:arg name="ros2_controllers_yaml" default=""/>
   <gazebo>
-    <plugin filename="libgazebo_ros2_control.so" name="gazebo_ros2_control">
+    <plugin filename="gz_ros2_control-system" name="gz_ros2_control::GzRos2ControlPlugin">
       <robot_param>robot_description</robot_param>
       <robot_param_node>robot_state_publisher</robot_param_node>
@@ -69,25 +69,46 @@
     </plugin>
   </gazebo>
-  <!-- Physics materials -->
+  <!-- Visual materials (Gz Sim uses explicit RGBA, not named Gazebo/ materials) -->
   <gazebo reference="base_link">
-    <material>Gazebo/Grey</material>
+    <material>
+      <ambient>0.4 0.4 0.4 1</ambient>
+      <diffuse>0.5 0.5 0.5 1</diffuse>
+    </material>
   </gazebo>
   <gazebo reference="link_1">
-    <material>Gazebo/Orange</material>
+    <material>
+      <ambient>0.9 0.5 0.0 1</ambient>
+      <diffuse>1.0 0.6 0.0 1</diffuse>
+    </material>
   </gazebo>
   <gazebo reference="link_2">
-    <material>Gazebo/Orange</material>
+    <material>
+      <ambient>0.9 0.5 0.0 1</ambient>
+      <diffuse>1.0 0.6 0.0 1</diffuse>
+    </material>
   </gazebo>
   <gazebo reference="link_3">
-    <material>Gazebo/Orange</material>
+    <material>
+      <ambient>0.9 0.5 0.0 1</ambient>
+      <diffuse>1.0 0.6 0.0 1</diffuse>
+    </material>
   </gazebo>
   <gazebo reference="link_4">
-    <material>Gazebo/Orange</material>
+    <material>
+      <ambient>0.9 0.5 0.0 1</ambient>
+      <diffuse>1.0 0.6 0.0 1</diffuse>
+    </material>
   </gazebo>
   <gazebo reference="link_5">
-    <material>Gazebo/Orange</material>
+    <material>
+      <ambient>0.9 0.5 0.0 1</ambient>
+      <diffuse>1.0 0.6 0.0 1</diffuse>
+    </material>
   </gazebo>
   <gazebo reference="link_6">
-    <material>Gazebo/Grey</material>
+    <material>
+      <ambient>0.4 0.4 0.4 1</ambient>
+      <diffuse>0.5 0.5 0.5 1</diffuse>
+    </material>
   </gazebo>
 </robot>
