Commit message: updated f/t sensor

File: kuka_refuel_ws/src/ur_description/urdf/ur5.urdf (robot description, URDF)
Before this commit: robot ur5_robot, 12 links, 11 joints
Links:
- added link ft_sensor_link, mass 0.05; visual cylinder length=0.005 radius=0.03
Joints:
- added joint ft_sensor_joint: type fixed, parent wrist_3_link, child ft_sensor_link, origin xyz=0 0 0 rpy=0 0 0
- joint wrist_3-flange: parent wrist_3_link -> ft_sensor_link
