Commit message: Fix: resolve mesh paths in KR8 URDF (remove xacro variables)

File: kuka_refuel_ws/src/kuka_kr6_gazebo/models/kr8_r2100/model.urdf (robot description, URDF)
Before this commit: robot kuka_kr8_r2100, 10 links, 9 joints
Links:
- link ${prefix}base_link: geometry collision mesh filename=meshes/collision/base_link.stl; visual mesh filename=meshes/visual/base_link.dae
- link ${prefix}link_1: geometry collision mesh filename=meshes/collision/link_1.stl; visual mesh filename=meshes/visual/link_1.dae
- link ${prefix}link_2: geometry collision mesh filename=meshes/collision/link_2.stl; visual mesh filename=meshes/visual/link_2.dae
- link ${prefix}link_3: geometry collision mesh filename=meshes/collision/link_3.stl; visual mesh filename=meshes/visual/link_3.dae
- link ${prefix}link_4: geometry collision mesh filename=meshes/collision/link_4.stl; visual mesh filename=meshes/visual/link_4.dae
- link ${prefix}link_5: geometry collision mesh filename=meshes/collision/link_5.stl; visual mesh filename=meshes/visual/link_5.dae
- link ${prefix}link_6: geometry collision mesh filename=meshes/collision/link_6.stl; visual mesh filename=meshes/visual/link_6.dae
